File: hardware/supply.kicad_sch (KiCad schematic)
At the start: 17 parts, among them U1 LM7805, U3 LM7812_TO220

Commit message: adicionando gerbers e atualização
Parts:
- R3: value 10k -> 20k
Changed lines of the file:
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@@
 		(fields_autoplaced yes)
 		(property "Reference" "R3"
-			(at 86.106 136.6519 0)
+			(at 86.36 136.6519 0)
 			(effects
 				(font
@@
 			)
 		)
-		(property "Value" "10k"
-			(at 86.106 139.1919 0)
+		(property "Value" "20k"
+			(at 86.36 139.1919 0)
 			(effects
 				(font
