File: hardware/MCU.kicad_sch (KiCad schematic)
At the start: 13 parts, among them J401 USART, U4 ATmega328P-P, Y401 16MHz

Commit message: adicionando arquivos
Parts:
- added D8: LED_RED, LED_SMD:LED_0805_2012Metric_Pad1.15x1.40mm_HandSolder, symbol Device:LED_Small
- added R16: 330, Resistor_SMD:R_0805_2012Metric_Pad1.20x1.40mm_HandSolder, symbol Device:R_Small
Connections:
- net GND: now also D8.1 (K)
- net at U4.28 (PC5): now also R16.1
- new net: D8.2 (A), R16.2
- no-connect marks 13 -> 12
Changed lines of the file:
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@@
+	)
+	(junction
+		(at 113.792 141.986)
+		(diameter 0)
+		(color 0 0 0 0)
 	)
 	(junction
@@
 	)
 	(no_connect
-		(at 129.032 102.616)
-	)
-	(no_connect
 		(at 129.032 92.456)
 	)
@@
 	(wire
 		(pts
+			(xy 145.796 102.616) (xy 145.796 131.191)
+		)
+		(stroke
+			(width 0)
+			(type default)
+		)
+	)
+	(wire
+		(pts
 			(xy 131.572 112.776) (xy 129.032 112.776)
 		)
@@
 	(wire
 		(pts
+			(xy 113.792 141.986) (xy 113.792 144.272)
+		)
+		(stroke
+			(width 0)
+			(type default)
+		)
+	)
+	(wire
+		(pts
 			(xy 163.322 105.156) (xy 155.067 105.156)
 		)
@@
 	(wire
 		(pts
+			(xy 129.032 102.616) (xy 145.796 102.616)
+		)
+		(stroke
+			(width 0)
+			(type default)
+		)
+	)
+	(wire
+		(pts
 			(xy 167.132 77.216) (xy 129.032 77.216)
 		)
@@
 	(wire
 		(pts
+			(xy 145.796 136.271) (xy 145.796 136.906)
+		)
+		(stroke
+			(width 0)
+			(type default)
+		)
+	)
+	(wire
+		(pts
 			(xy 207.772 98.806) (xy 207.772 96.266)
 		)
@@
 	(wire
 		(pts
-			(xy 113.792 135.636) (xy 113.792 140.716)
+			(xy 113.792 135.636) (xy 113.792 141.986)
 		)
 		(stroke
@@
 		(pts
 			(xy 129.032 84.836) (xy 207.772 84.836)
+		)
+		(stroke
+			(width 0)
+			(type default)
+		)
+	)
+	(wire
+		(pts
+			(xy 113.792 141.986) (xy 145.796 141.986)
 		)
 		(stroke
@@
 	(symbol
 		(lib_id "power:GND")
-		(at 113.792 140.716 0)
+		(at 113.792 144.272 0)
 		(unit 1)
 		(exclude_from_sim no)
@@
 		(dnp no)
 		(property "Reference" "#PWR0412"
-			(at 113.792 147.066 0)
+			(at 113.792 150.622 0)
 			(effects
 				(font
@@
 		)
 		(property "Value" "GND"
-			(at 115.062 145.796 0)
+			(at 115.062 149.352 0)
 			(effects
 				(font
@@
 		)
 		(property "Footprint" ""
-			(at 113.792 140.716 0)
+			(at 113.792 144.272 0)
 			(effects
 				(font
@@
 		)
 		(property "Datasheet" ""
-			(at 113.792 140.716 0)
+			(at 113.792 144.272 0)
 			(effects
 				(font
@@
 		)
 		(property "Description" ""
-			(at 113.792 140.716 0)
+			(at 113.792 144.272 0)
 			(effects
 				(font
@@
 	)
 	(symbol
+		(lib_id "Device:LED_Small")
+		(at 145.796 139.446 90)
+		(unit 1)
+		(exclude_from_sim no)
+		(in_bom yes)
+		(on_board yes)
+		(dnp no)
+		(property "Reference" "D8"
+			(at 150.241 141.351 0)
+			(effects
+				(font
+					(size 1.27 1.27)
+				)
+				(justify left)
+			)
+		)
+		(property "Value" "LED_RED"
+			(at 148.336 141.986 0)
+			(effects
+				(font
+					(size 1.27 1.27)
+				)
+				(justify left)
+			)
+		)
+		(property "Footprint" "LED_SMD:LED_0805_2012Metric_Pad1.15x1.40mm_HandSolder"
+			(at 145.796 139.446 90)
+			(effects
+				(font
+					(size 1.27 1.27)
+				)
+				(hide yes)
+			)
+		)
+		(property "Datasheet" ""
+			(at 145.796 139.446 90)
+			(effects
+				(font
+					(size 1.27 1.27)
+				)
+				(hide yes)
+			)
+		)
+		(property "Description" ""
+			(at 145.796 139.446 0)
+			(effects
+				(font
+					(size 1.27 1.27)
+				)
+				(hide yes)
+			)
+		)
+		(pin "1"
+		)
+		(pin "2"
+		)
+		(instances
+			(project "MSC25"
+				(path "/54fa0170-a23b-4b64-b583-87dd15942089/720cf98c-f22b-4ae7-9df1-2d7e833b78e5"
+					(reference "D8")
+					(unit 1)
+				)
+			)
+		)
+	)
+	(symbol
 		(lib_id "MCU_Microchip_ATmega:ATmega328P-P")
 		(at 113.792 97.536 0)
@@
 					(unit 1)
 				)
+			)
+		)
+	)
+	(symbol
+		(lib_id "Device:R_Small")
+		(at 145.796 133.731 0)
+		(unit 1)
+		(exclude_from_sim no)
+		(in_bom yes)
+		(on_board yes)
+		(dnp no)
+		(property "Reference" "R16"
+			(at 147.701 128.016 90)
+			(effects
+				(font
+					(size 1.27 1.27)
+				)
+			)
+		)
+		(property "Value" "330"
+			(at 143.764 133.604 90)
+			(effects
+				(font
+					(size 1.27 1.27)
+				)
+			)
+		)
+		(property "Footprint" "Resistor_SMD:R_0805_2012Metric_Pad1.20x1.40mm_HandSolder"
+			(at 145.796 133.731 0)
+			(effects
+				(font
+					(size 1.27 1.27)
+				)
+				(hide yes)
+			)
+		)
+		(property "Datasheet" "~"
+			(at 145.796 133.731 0)
+			(effects
+				(font
+					(size 1.27 1.27)
+				)
+				(hide yes)
+			)
+		)
+		(property "Description" ""
+			(at 145.796 133.731 0)
+			(effects
+				(font
+					(size 1.27 1.27)
+				)
+				(hide yes)
+			)
+		)
+		(pin "1"
+		)
+		(pin "2"
+		)
+		(instances
+			(project "MSC25"
+				(path "/54fa0170-a23b-4b64-b583-87dd15942089/720cf98c-f22b-4ae7-9df1-2d7e833b78e5"
+					(reference "R16")
+					(unit 1)
+				)

Commit message: atualizações
Parts:
- U4: footprint Package_DIP:DIP-28_W7.62mm -> Package_DIP:DIP-28_W7.62mm_LongPads
Changed lines of the file:
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@@
 			)
 		)
-		(property "Footprint" "Package_DIP:DIP-28_W7.62mm"
+		(property "Footprint" "Package_DIP:DIP-28_W7.62mm_LongPads"
 			(at 113.792 97.536 0)
 			(effects
