File: hardware/MSC25.kicad_pcb (KiCad board)
At the start: 2 copper layers, 63 x 108 mm, 58 parts, among them J1 Sensor_I, J401 USART, J601 RJ45, J602 RJ45, U1 LM7805, U2 LM324, U201 MCP2551-I/SN, U202 MCP2515-xSO, U3 LM7812_TO220, U4 ATmega328P-P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

Commit message: adicionando arquivos
Parts:
- added D8: LED_RED, LED_SMD:LED_0805_2012Metric_Pad1.15x1.40mm_HandSolder, F.Cu at (132.8, 112.0)
- added R16: 330, Resistor_SMD:R_0805_2012Metric_Pad1.20x1.40mm_HandSolder, F.Cu at (135.8, 112.0)
Connections:
- PS1 pad 3: -15V -> +15V
- PS501 pad 4: +15V -> -15V
- U4 pad 28: unconnected-(U4-PC5-Pad28) -> Net-(U4-PC5)
Routing:
- net Net-(U4-PC5): track 0.00 -> 36.1 mm
- net Net-(D8-A): track 0.00 -> 3.07 mm

Commit message: adicionando gerbers e atualização
Parts:
- R3: value 10k -> 20k
Changed lines of the file:
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@@
 			)
 		)
-		(property "Value" "10k"
+		(property "Value" "20k"
 			(at 0 -1.65 90)
 			(layer "B.Fab")

Commit message: atualizações
Parts:
- added D3: 5V, Diode_SMD:D_MiniMELF, F.Cu at (162.4, 108.4)
- C401, C402: moved to B.Cu
- U4: footprint Package_DIP:DIP-28_W7.62mm -> Package_DIP:DIP-28_W7.62mm_LongPads
- moved D8 29.3 mm to (161.4, 118.2)
- moved R16 29.3 mm to (164.5, 118.2)
- moved C401 7.15 mm to (173.0, 101.6), turned to 0 degrees
- moved C402 7.13 mm to (173.0, 98.8), turned to 180 degrees
- moved R1 6.38 mm to (153.9, 98.6)
- moved C404 4.25 mm to (186.8, 99.2), turned to 0 degrees
Connections:
- PS1 pad 3: +15V -> -15V
- PS501 pad 4: -15V -> +15V
- R1 pad 2: Net-(U2A-+) -> Net-(U2A--)
- R2 pad 1: Net-(U2A-+) -> Net-(U2A--)
- R2 pad 2: Net-(U2B--) -> Net-(U2B-+)
- U2 pad 1: Net-(U2B--) -> Net-(U2B-+)
- U2 pad 2: +1,67V -> Net-(U2A--)
- U2 pad 3: Net-(U2A-+) -> +1,67V
- U2 pad 5: /Analog/S -> Net-(U2B-+)
- U2 pad 6: Net-(U2B--) -> /Analog/S
Routing:
- net Net-(U4-PC5): track 36.1 -> 4.81 mm
- net Net-(U2B--): track 18.8 -> 0.00 mm
- net Net-(U2B-+): track 0.00 -> 18.5 mm
- net Net-(U2A--): track 0.00 -> 7.80 mm
- net Net-(U2A-+): track 7.35 -> 0.00 mm
- net +1,67V: track 13.8 -> 16.5 mm
- net -15V: track 16.8 -> 15.0 mm
- net /Analog/OUT: track 19.0 -> 17.6 mm
- net +5V: track 175.5 -> 174.2 mm
- net Net-(U4-XTAL1/PB6): track 9.50 -> 8.95 mm
- net GND: vias 1 -> 15
