File: hardware/MSC25.kicad_sch (KiCad schematic)
At the start: 1 part, among them J1 Sensor_I

Commit message: atualizações
Changed lines of the file:
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@@
+	(wire
+		(pts
+			(xy 152.654 78.232) (xy 154.686 78.232)
+		)
+		(stroke
+			(width 0)
+			(type default)
+		)
+	)
+	(wire
+		(pts
+			(xy 70.358 33.782) (xy 76.454 33.782)
+		)
+		(stroke
+			(width 0)
+			(type default)
+		)
+	)
+	(wire
+		(pts
+			(xy 68.326 78.994) (xy 68.326 33.782)
+		)
+		(stroke
+			(width 0)
+			(type default)
+		)
+	)
+	(wire
+		(pts
+			(xy 50.546 29.21) (xy 76.454 29.21)
+		)
+		(stroke
+			(width 0)
+			(type default)
+		)
+	)
+	(wire
+		(pts
+			(xy 66.294 81.28) (xy 76.454 81.28)
+		)
+		(stroke
+			(width 0)
+			(type default)
+		)
+	)
+	(wire
+		(pts
+			(xy 188.722 74.93) (xy 188.722 76.2)
+		)
+		(stroke
+			(width 0)
+			(type default)
+		)
+	)
 	(wire
 		(pts
@@
 	(wire
 		(pts
-			(xy 70.358 33.782) (xy 76.454 33.782)
-		)
-		(stroke
-			(width 0)
-			(type default)
-		)
-	)
-	(wire
-		(pts
-			(xy 68.326 78.994) (xy 68.326 33.782)
-		)
-		(stroke
-			(width 0)
-			(type default)
-		)
-	)
-	(wire
-		(pts
-			(xy 50.546 29.21) (xy 76.454 29.21)
-		)
-		(stroke
-			(width 0)
-			(type default)
-		)
-	)
-	(wire
-		(pts
-			(xy 66.294 81.28) (xy 76.454 81.28)
-		)
-		(stroke
-			(width 0)
-			(type default)
-		)
-	)
-	(wire
-		(pts
-			(xy 188.722 74.93) (xy 188.722 76.2)
-		)
-		(stroke
-			(width 0)
-			(type default)
-		)
-	)
-	(wire
-		(pts
-			(xy 152.654 78.232) (xy 154.686 78.232)
-		)
-		(stroke
-			(width 0)
-			(type default)
-		)
-	)
-	(wire
-		(pts
 			(xy 101.346 80.264) (xy 127 80.264)
 		)
@@
 	(wire
 		(pts
-			(xy 101.346 31.496) (xy 104.14 31.496)
+			(xy 101.346 31.496) (xy 105.918 31.496)
 		)
 		(stroke
@@
 	(wire
 		(pts
-			(xy 101.346 34.036) (xy 104.14 34.036)
-		)
-		(stroke
-			(width 0)
-			(type default)
-		)
-	)
-	(wire
-		(pts
 			(xy 194.31 74.93) (xy 194.31 76.2)
 		)
@@
 		(pts
 			(xy 70.358 33.782) (xy 70.358 35.814)
+		)
+		(stroke
+			(width 0)
+			(type default)
+		)
+	)
+	(wire
+		(pts
+			(xy 105.41 34.036) (xy 101.346 34.036)
 		)
 		(stroke
@@
 	(symbol
 		(lib_id "power:+15V")
-		(at 104.14 34.036 270)
+		(at 105.918 31.496 270)
 		(unit 1)
 		(exclude_from_sim no)
@@
 		(fields_autoplaced yes)
 		(property "Reference" "#PWR016"
-			(at 100.33 34.036 0)
+			(at 102.108 31.496 0)
 			(effects
 				(font
@@
 		)
 		(property "Value" "+15V"
-			(at 108.458 34.0359 90)
+			(at 110.236 31.4959 90)
 			(effects
 				(font
@@
 		)
 		(property "Footprint" ""
-			(at 104.14 34.036 0)
+			(at 105.918 31.496 0)
 			(effects
 				(font
@@
 		)
 		(property "Datasheet" ""
-			(at 104.14 34.036 0)
+			(at 105.918 31.496 0)
 			(effects
 				(font
@@
 		)
 		(property "Description" "Power symbol creates a global label with name \"+15V\""
-			(at 104.14 34.036 0)
+			(at 105.918 31.496 0)
 			(effects
 				(font
@@
 	(symbol
 		(lib_id "power:GND")
-		(at 154.686 78.232 180)
+		(at 154.686 80.264 0)
+		(mirror y)
 		(unit 1)
 		(exclude_from_sim no)
@@
 		(fields_autoplaced yes)
 		(property "Reference" "#PWR011"
-			(at 154.686 71.882 0)
+			(at 154.686 86.614 0)
 			(effects
 				(font
@@
 		)
 		(property "Value" "GND"
-			(at 154.686 73.66 0)
+			(at 154.686 84.836 0)
 			(effects
 				(font
@@
 		)
 		(property "Footprint" ""
-			(at 154.686 78.232 0)
+			(at 154.686 80.264 0)
 			(effects
 				(font
@@
 		)
 		(property "Datasheet" ""
-			(at 154.686 78.232 0)
+			(at 154.686 80.264 0)
 			(effects
 				(font
@@
 		)
 		(property "Description" "Power symbol creates a global label with name \"GND\" , ground"
-			(at 154.686 78.232 0)
+			(at 154.686 80.264 0)
 			(effects
 				(font
@@
 	(symbol
 		(lib_id "power:+5V")
-		(at 154.686 80.264 180)
+		(at 154.686 78.232 0)
+		(mirror y)
 		(unit 1)
 		(exclude_from_sim no)
@@
 		(fields_autoplaced yes)
 		(property "Reference" "#PWR013"
-			(at 154.686 76.454 0)
+			(at 154.686 82.042 0)
 			(effects
 				(font
@@
 		)
 		(property "Value" "+5V"
-			(at 154.686 84.836 0)
+			(at 154.686 73.66 0)
 			(effects
 				(font
@@
 		)
 		(property "Footprint" ""
-			(at 154.686 80.264 0)
+			(at 154.686 78.232 0)
 			(effects
 				(font
@@
 		)
 		(property "Datasheet" ""
-			(at 154.686 80.264 0)
+			(at 154.686 78.232 0)
 			(effects
 				(font
@@
 		)
 		(property "Description" "Power symbol creates a global label with name \"+5V\""
-			(at 154.686 80.264 0)
+			(at 154.686 78.232 0)
 			(effects
 				(font
@@
 	(symbol
 		(lib_id "power:-15V")
-		(at 104.14 31.496 270)
+		(at 105.41 34.036 270)
 		(unit 1)
 		(exclude_from_sim no)
@@
 		(fields_autoplaced yes)
 		(property "Reference" "#PWR015"
-			(at 100.33 31.496 0)
+			(at 101.6 34.036 0)
 			(effects
 				(font
@@
 		)
 		(property "Value" "-15V"
-			(at 108.458 31.4959 90)
+			(at 109.728 34.0359 90)
 			(effects
 				(font
@@
 		)
 		(property "Footprint" ""
-			(at 104.14 31.496 0)
+			(at 105.41 34.036 0)
 			(effects
 				(font
@@
 		)
 		(property "Datasheet" ""
-			(at 104.14 31.496 0)
+			(at 105.41 34.036 0)
 			(effects
 				(font
@@
 		)
 		(property "Description" "Power symbol creates a global label with name \"-15V\""
-			(at 104.14 31.496 0)
+			(at 105.41 34.036 0)
 			(effects
 				(font
@@
 		)
 		(instances
-			(project ""
+			(project "MSC25"
 				(path "/54fa0170-a23b-4b64-b583-87dd15942089"
 					(reference "#PWR015")
@@
 		)
 		(pin "GND" output
-			(at 152.654 78.232 0)
+			(at 152.654 80.264 0)
 			(effects
 				(font
@@
 		)
 		(pin "VCC" input
-			(at 152.654 80.264 0)
-			(effects
-				(font
+			(at 152.654 78.232 0)
+			(effects
+				(font
