File: hardware/analog.kicad_sch (KiCad schematic)
At the start: 4 parts, among them U2 LM324

Commit message: atualizações
Parts:
- added D3: 5V, Diode_SMD:D_MiniMELF, symbol Módulo-temperatura-rescue:D_Zener_Small-Device
Connections:
- net 1.67V: now also U2.3 (+); no longer U2.2 (-)
- net GND: now also D3.2 (A)
- net S: now also U2.6 (-), D3.1 (K); no longer U2.5 (+)
- net at R1.2, R2.1: now also U2.2 (-); no longer U2.3 (+)
- net at R2.2, U2.1: now also U2.5 (+); no longer U2.6 (-)
Changed lines of the file:
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@@
+	)
+	(junction
+		(at 138.684 57.404)
+		(diameter 0)
+		(color 0 0 0 0)
 	)
 	(junction
@@
 	(wire
 		(pts
+			(xy 138.684 58.928) (xy 138.684 57.404)
+		)
+		(stroke
+			(width 0)
+			(type default)
+		)
+	)
+	(wire
+		(pts
 			(xy 94.488 45.466) (xy 94.488 57.404)
 		)
@@
 	(wire
 		(pts
+			(xy 138.684 64.008) (xy 138.684 66.04)
+		)
+		(stroke
+			(width 0)
+			(type default)
+		)
+	)
+	(wire
+		(pts
 			(xy 85.598 77.724) (xy 95.504 77.724)
 		)
@@
 	(wire
 		(pts
+			(xy 138.684 57.404) (xy 142.494 57.404)
+		)
+		(stroke
+			(width 0)
+			(type default)
+		)
+	)
+	(wire
+		(pts
 			(xy 134.874 48.768) (xy 134.874 57.404)
 		)
@@
 	(wire
 		(pts
-			(xy 134.874 57.404) (xy 138.176 57.404)
+			(xy 134.874 57.404) (xy 138.684 57.404)
 		)
 		(stroke
@@
 	(hierarchical_label "S"
 		(shape input)
-		(at 138.176 57.404 0)
+		(at 142.494 57.404 0)
 		(effects
 			(font
@@
 	)
 	(symbol
+		(lib_id "Módulo-temperatura-rescue:D_Zener_Small-Device")
+		(at 138.684 61.468 270)
+		(unit 1)
+		(exclude_from_sim no)
+		(in_bom yes)
+		(on_board yes)
+		(dnp no)
+		(property "Reference" "D3"
+			(at 140.97 61.468 0)
+			(effects
+				(font
+					(size 1.27 1.27)
+				)
+			)
+		)
+		(property "Value" "5V"
+			(at 136.398 61.468 0)
+			(effects
+				(font
+					(size 1.27 1.27)
+				)
+			)
+		)
+		(property "Footprint" "Diode_SMD:D_MiniMELF"
+			(at 138.684 61.468 90)
+			(effects
+				(font
+					(size 1.27 1.27)
+				)
+				(hide yes)
+			)
+		)
+		(property "Datasheet" ""
+			(at 138.684 61.468 90)
+			(effects
+				(font
+					(size 1.27 1.27)
+				)
+				(hide yes)
+			)
+		)
+		(property "Description" ""
+			(at 138.684 61.468 0)
+			(effects
+				(font
+					(size 1.27 1.27)
+				)
+			)
+		)
+		(pin "1"
+		)
+		(pin "2"
+		)
+		(instances
+			(project "MSC25"
+				(path "/54fa0170-a23b-4b64-b583-87dd15942089/6a4927c6-3e9d-481f-a7c7-87205ab2eb3d"
+					(reference "D3")
+					(unit 1)
+				)
+			)
+		)
+	)
+	(symbol
 		(lib_id "Amplifier_Operational:LM324")
 		(at 127.254 57.404 0)
+		(mirror x)
 		(unit 2)
 		(exclude_from_sim no)
@@
 		(on_board yes)
 		(dnp no)
-		(fields_autoplaced yes)
 		(property "Reference" "U2"
-			(at 127.254 47.498 0)
+			(at 127.254 67.31 0)
 			(effects
 				(font
@@
 		)
 		(property "Value" "LM324"
-			(at 127.254 50.038 0)
+			(at 127.254 64.77 0)
 			(effects
 				(font
@@
 		)
 		(property "Footprint" ""
-			(at 125.984 54.864 0)
+			(at 125.984 59.944 0)
 			(effects
 				(font
@@
 		)
 		(property "Datasheet" "http://www.ti.com/lit/ds/symlink/lm2902-n.pdf"
-			(at 128.524 52.324 0)
+			(at 128.524 62.484 0)
 			(effects
 				(font
@@
 		(lib_id "Amplifier_Operational:LM324")
 		(at 103.886 59.944 0)
+		(mirror x)
 		(unit 1)
 		(exclude_from_sim no)
@@
 		(on_board yes)
 		(dnp no)
-		(fields_autoplaced yes)
 		(property "Reference" "U2"
-			(at 103.886 49.53 0)
+			(at 103.886 70.358 0)
 			(effects
 				(font
@@
 		)
 		(property "Value" "LM324"
-			(at 103.886 52.07 0)
+			(at 103.886 67.818 0)
 			(effects
 				(font
@@
 		)
 		(property "Footprint" "Package_DIP:DIP-14_W7.62mm"
-			(at 102.616 57.404 0)
+			(at 102.616 62.484 0)
 			(effects
 				(font
@@
 		)
 		(property "Datasheet" "http://www.ti.com/lit/ds/symlink/lm2902-n.pdf"
-			(at 105.156 54.864 0)
+			(at 105.156 65.024 0)
 			(effects
 				(font
@@
 					(unit 1)
 				)
+			)
+		)
+	)
+	(symbol
+		(lib_id "power:GND")
+		(at 138.684 66.04 0)
+		(unit 1)
+		(exclude_from_sim no)
+		(in_bom yes)
+		(on_board yes)
+		(dnp no)
+		(fields_autoplaced yes)
+		(property "Reference" "#PWR029"
+			(at 138.684 72.39 0)
+			(effects
+				(font
+					(size 1.27 1.27)
+				)
+				(hide yes)
+			)
+		)
+		(property "Value" "GND"
+			(at 138.684 70.4834 0)
+			(effects
+				(font
+					(size 1.27 1.27)
+				)
+			)
+		)
+		(property "Footprint" ""
+			(at 138.684 66.04 0)
+			(effects
+				(font
+					(size 1.27 1.27)
+				)
+				(hide yes)
+			)
+		)
+		(property "Datasheet" ""
+			(at 138.684 66.04 0)
+			(effects
+				(font
+					(size 1.27 1.27)
+				)
+				(hide yes)
+			)
+		)
+		(property "Description" ""
+			(at 138.684 66.04 0)
+			(effects
+				(font
+					(size 1.27 1.27)
+				)
+			)
+		)
+		(pin "1"
+		)
+		(instances
+			(project "MSC25"
+				(path "/54fa0170-a23b-4b64-b583-87dd15942089/6a4927c6-3e9d-481f-a7c7-87205ab2eb3d"
+					(reference "#PWR029")
+					(unit 1)
+				)
